Commit message: using xacro for dynamically loading descriptions about grippers, added fingers and finger_tips to hand groups so grasping wouldn't considered as collision anymore

File: config/baxter.srdf.xacro (robot description, xacro)
@@ -3,4 +3,6 @@
   <xacro:arg name="left_tip_name" default="left_gripper"/>
   <xacro:arg name="right_tip_name" default="right_gripper"/>
+  <xacro:arg name="left_electric_gripper" default="false"/>
+  <xacro:arg name="right_electric_gripper" default="false"/>
   <xacro:include filename="$(find baxter_moveit_config)/config/baxter_base.srdf.xacro" />
   <xacro:baxter_base left_tip_name="$(arg left_tip_name)" right_tip_name="$(arg right_tip_name)"/>
@@ -8,5 +10,4 @@
   <xacro:include filename="$(find baxter_moveit_config)/config/default_gripper.srdf.xacro" />
   <xacro:default_gripper side="left"/>
-  <xacro:arg name="left_electric_gripper" default="false"/>
   <xacro:if value="$(arg left_electric_gripper)">
     <xacro:include filename="$(find baxter_moveit_config)/config/rethink_electric_gripper.srdf.xacro" />
@@ -16,5 +17,4 @@
   <xacro:include filename="$(find baxter_moveit_config)/config/default_gripper.srdf.xacro" />
   <xacro:default_gripper side="right"/>
-  <xacro:arg name="right_electric_gripper" default="false"/>
   <xacro:if value="$(arg right_electric_gripper)">
     <xacro:include filename="$(find baxter_moveit_config)/config/rethink_electric_gripper.srdf.xacro" />

File: config/baxter_base.srdf.xacro (robot description, xacro)
@@ -27,6 +27,12 @@
         <link name="left_gripper_base" />
         <link name="left_gripper" />
-	<joint name="l_gripper_l_finger_joint" />
-	<joint name="l_gripper_r_finger_joint" />
+	<xacro:if value="$(arg left_electric_gripper)">
+		<joint name="l_gripper_l_finger_joint" />
+		<joint name="l_gripper_r_finger_joint" />
+		<link name="l_gripper_l_finger_tip" />
+		<link name="l_gripper_l_finger" />
+		<link name="l_gripper_r_finger_tip" />
+		<link name="l_gripper_r_finger" />
+	</xacro:if>
     </group>
     <group name="right_hand">
@@ -34,6 +40,12 @@
         <link name="right_gripper_base" />
         <link name="right_gripper" />
-	<!--<joint name="r_gripper_l_finger_joint" />
-	<joint name="r_gripper_r_finger_joint" />-->
+	<xacro:if value="$(arg right_electric_gripper)">
+		<joint name="r_gripper_l_finger_joint" />
+		<joint name="r_gripper_r_finger_joint" />
+		<link name="r_gripper_l_finger_tip" />
+		<link name="r_gripper_l_finger" />
+		<link name="r_gripper_r_finger_tip" />
+		<link name="r_gripper_r_finger" />
+	</xacro:if>
     </group>
     <!--END EFFECTOR: Purpose: Represent information about an end effector.-->
